File: prozessorboard/processorboard_v3-1-1/CAN_connect.sch (KiCad schematic (older format))
At the start: 3 parts, among them U2 SN65HVD230

Commit message: Update github with current version of tera local
Parts:
- C17: symbol C_Small -> Device:C_Small
- R8: symbol R_Small -> Device:R_Small
- U2: symbol SN65HVD230 -> tera_logic:SN65HVD230
Changed lines of the file:
@@
-EESchema Schematic File Version 2
-LIBS:power
-LIBS:device
-LIBS:transistors
-LIBS:conn
-LIBS:linear
-LIBS:regul
-LIBS:74xx
-LIBS:cmos4000
-LIBS:adc-dac
-LIBS:memory
-LIBS:xilinx
-LIBS:microcontrollers
-LIBS:dsp
-LIBS:microchip
-LIBS:analog_switches
-LIBS:motorola
-LIBS:texas
-LIBS:intel
-LIBS:audio
-LIBS:interface
-LIBS:digital-audio
-LIBS:philips
-LIBS:display
-LIBS:cypress
-LIBS:siliconi
-LIBS:opto
-LIBS:atmel
-LIBS:contrib
-LIBS:valves
-LIBS:ft232rl
-LIBS:relais
-LIBS:Supply
-LIBS:tera_general
-LIBS:tera_logic
-LIBS:tera_processors
-LIBS:tera_switches
-LIBS:local_pwr
-LIBS:tera_connectors
-LIBS:tera_emc_prodection
-LIBS:local_special
+EESchema Schematic File Version 4
 LIBS:stm32f4-board_v3-x-cache
-EELAYER 25 0
+EELAYER 26 0
 EELAYER END
 $Descr A4 11693 8268
@@
 $EndSheet
 $Comp
-L SN65HVD230 U2
+L tera_logic:SN65HVD230 U2
 U 1 1 57F8E8FC
 P 6050 3300
@@
 $EndComp
 $Comp
-L C_Small C17
+L Device:C_Small C17
 U 1 1 57F91A9B
 P 5200 2950
@@
 $EndComp
 $Comp
-L R_Small R8
+L Device:R_Small R8
 U 1 1 580DEA21
 P 4950 3400
@@
 GND
 Wire Wire Line
-	5600 1500 5600 1500
-Wire Wire Line
 	4700 3200 5550 3200
 Wire Wire Line
@@
 	5150 3050 5200 3050
 Wire Wire Line
-	5150 2850 5550 2850
+	5150 2850 5200 2850
 Wire Wire Line
 	5550 2850 5550 3100
@@
 Connection ~ 5200 2850
 NoConn ~ 6550 3100
+Wire Wire Line
+	5200 2850 5550 2850
 $EndSCHEMATC
