File: prozessorboard/processorboard_v3-1-1/stm32f4-board_v3-x.kicad_pcb (KiCad board)
At the start: 4 copper layers, 51 x 33 mm, 87 parts, among them IC1 LM4132A-3.3, P1 Left, P2 Right, P3 TERA_Debug_14pol, P4 CAN_CON_2pol, U1 STM32-F405RGT6, U2 SN65HVD230, U3 SN65HVD230, Y1 8MHz, x1 gnd_contact, x12 gnd_contact, x15 gnd_contact, x2 gnd_contact, x3 gnd_contact, x4 gnd_contact, x5 gnd_contact, x6 gnd_contact, x7 gnd_contact, x8 gnd_contact, x9 gnd_contact

Commit message: Update github with current version of tera local
Changed lines of the file:
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@@
-(kicad_pcb (version 4) (host pcbnew no-vcs-found-product)
+(kicad_pcb (version 20171130) (host pcbnew 6.0.0-rc1-unknown-r13958-f11cb736)
   (general
-    (links 236)
-    (no_connects 0)
-    (area 86 98.8 165.285716 154.245001)
     (thickness 1.6)
     (drawings 29)
@@
     (zone_45_only yes)
     (trace_min 0.2)
-    (segment_width 0.2)
-    (edge_width 0.15)
     (via_size 0.65)
     (via_drill 0.2)
@@
     (uvia_min_size 0.2)
     (uvia_min_drill 0.1)
+    (edge_width 0.15)
+    (segment_width 0.2)
     (pcb_text_width 0.3)
     (pcb_text_size 1.5 1.5)
@@
       (layerselection 0x010f0_ffffffff)
       (usegerberextensions false)
+      (usegerberattributes false)
+      (usegerberadvancedattributes false)
+      (creategerberjobfile false)
       (excludeedgelayer true)
       (linewidth 0.100000)
@@
       (hpglpennumber 1)
       (hpglpenspeed 20)
-      (hpglpendiameter 15)
+      (hpglpendiameter 15.000000)
       (psnegative false)
       (psa4output false)
@@
       (drillshape 0)
       (scaleselection 1)
-      (outputdirectory gerber/))
+      (outputdirectory "gerber/"))
   )
   (net 0 "")
@@
     (attr smd)
     (fp_text reference svg2mod (at 0 -4.45995) (layer F.SilkS) hide
-      (effects (font (thickness 0.3048)))
+      (effects (font (size 1.524 1.524) (thickness 0.3048)))
     )
     (fp_text value G*** (at 0 4.45995) (layer F.SilkS) hide
-      (effects (font (thickness 0.3048)))
+      (effects (font (size 1.524 1.524) (thickness 0.3048)))
     )
     (fp_poly (pts (xy 4.627814 -0.545546) (xy 4.638286 -0.52065) (xy 4.64539 -0.492767) (xy 4.649629 -0.462455)
@@
       (xy 1.511193 -0.338215) (xy 1.50027 -0.299231) (xy 1.493022 -0.270419) (xy 1.490395 -0.259173)
       (xy 1.278209 0.543811) (xy 1.253249 0.647821) (xy 1.229813 0.767152) (xy 1.223474 0.794555)
-      (xy 1.219993 0.811475) (xy 1.219993 0.811475)) (layer F.SilkS) (width 0))
+      (xy 1.219993 0.811475)) (layer F.SilkS) (width 0))
   )
   (module tera_logos:TERA_Logo_SilkS_5x12.5mm locked (layer B.Cu)
@@
     (attr smd)
     (fp_text reference svg2mod (at 0 5.714667 180) (layer B.SilkS) hide
-      (effects (font (thickness 0.3048)) (justify mirror))
+      (effects (font (size 1.524 1.524) (thickness 0.3048)) (justify mirror))
     )
     (fp_text value G*** (at 0 -5.714667 180) (layer B.SilkS) hide
-      (effects (font (thickness 0.3048)) (justify mirror))
+      (effects (font (size 1.524 1.524) (thickness 0.3048)) (justify mirror))
     )
     (fp_poly (pts (xy -0.000023 2.666667) (xy -0.000023 2.400911) (xy 0.040353 2.400866) (xy 0.080672 2.400733)
