File: prozessorboard/processorboard_v3-1-1/stm32f4-board_v3-x.sch (KiCad schematic (older format))
At the start: 47 parts, among them P1 Left, P2 Right, P3 TERA_Debug_14pol, U1 STM32-F405RGT6, Y1 8MHz, x1 gnd_contact, x12 gnd_contact, x15 gnd_contact, x2 gnd_contact, x3 gnd_contact, x4 gnd_contact, x5 gnd_contact, x6 gnd_contact, x7 gnd_contact, x8 gnd_contact, x9 gnd_contact

Commit message: Update github with current version of tera local
Parts:
- C1, C10, C11, C12, C14, C16, C2, C3, C4, C5, C6, C7, C8, C9: symbol C_Small -> Device:C_Small
- D1, D2, D3: symbol Led_Small -> Device:LED_Small
- JP1, JP10, JP11, JP2, JP3, JP5, JP6, JP9: symbol Jumper_NO_Small -> Device:Jumper_NO_Small
- P1, P2: symbol ConnHirose_DF17-40DX-0.5V -> tera_connectors:ConnHirose_DF17-40DX-0.5V
- P3: symbol TERA_Debug_14pol -> tera_connectors:TERA_Debug_14pol
- R1, R2, R3, R4, R5: symbol R_Small -> Device:R_Small
- S2: symbol Button_NO_01x02 -> tera_switches:Button_NO_01x02
- U1: symbol STM32-F405RGT6 -> tera_processors:STM32-F405RGT6
- Y1: symbol Crystal_Small -> Device:Crystal_Small
- x1, x12, x15, x2, x3, x4, x5, x6, x7, x8, x9: symbol gnd_contact -> local_special:gnd_contact
