File: prozessorboard/processorboard_v3-1-1/supply.sch (KiCad schematic (older format))
At the start: 17 parts, among them IC1 LM4132A-3.3, U1 STM32-F405RGT6

Commit message: Update github with current version of tera local
Parts:
- C18, C24, C27, C28: symbol CP_Small -> Device:CP_Small
- C19, C20, C21, C22, C25, C26: symbol C_Small -> Device:C_Small
- D18, D19: symbol Led_Small -> Device:LED_Small
- IC1: symbol LM4132A-3.3 -> Supply:LM4132A-3.3
- JP4: symbol Jumper_NO_Small -> Device:Jumper_NO_Small
- R6, R7: symbol R_Small -> Device:R_Small
- U1: symbol STM32-F405RGT6 -> tera_processors:STM32-F405RGT6
Changed lines of the file:
@@
-EESchema Schematic File Version 2
-LIBS:power
-LIBS:device
-LIBS:transistors
-LIBS:conn
-LIBS:linear
-LIBS:regul
-LIBS:74xx
-LIBS:cmos4000
-LIBS:adc-dac
-LIBS:memory
-LIBS:xilinx
-LIBS:microcontrollers
-LIBS:dsp
-LIBS:microchip
-LIBS:analog_switches
-LIBS:motorola
-LIBS:texas
-LIBS:intel
-LIBS:audio
-LIBS:interface
-LIBS:digital-audio
-LIBS:philips
-LIBS:display
-LIBS:cypress
-LIBS:siliconi
-LIBS:opto
-LIBS:atmel
-LIBS:contrib
-LIBS:valves
-LIBS:ft232rl
-LIBS:relais
-LIBS:Supply
-LIBS:tera_general
-LIBS:tera_logic
-LIBS:tera_processors
-LIBS:tera_switches
-LIBS:local_pwr
-LIBS:tera_connectors
-LIBS:tera_emc_prodection
-LIBS:local_special
+EESchema Schematic File Version 4
 LIBS:stm32f4-board_v3-x-cache
-EELAYER 25 0
+EELAYER 26 0
 EELAYER END
 $Descr A4 11693 8268
@@
 $EndDescr
 $Comp
-L STM32-F405RGT6 U?
+L tera_processors:STM32-F405RGT6 U?
 U 8 1 57F984A6
 P 3300 4500
@@
 $EndComp
 $Comp
-L C_Small C25
+L Device:C_Small C25
 U 1 1 57FCAECB
 P 2900 3400
@@
 $EndComp
 $Comp
-L C_Small C26
+L Device:C_Small C26
 U 1 1 57FCCA2C
 P 2900 4900
@@
 $EndComp
 $Comp
-L C_Small C22
+L Device:C_Small C22
 U 1 1 57FCDD54
 P 2650 4900
@@
 $EndComp
 $Comp
-L C_Small C20
+L Device:C_Small C20
 U 1 1 57FCDDEB
 P 2350 4900
@@
 $EndComp
 $Comp
-L C_Small C19
+L Device:C_Small C19
 U 1 1 57FCDE81
 P 2100 4900
@@
 $EndComp
 $Comp
-L C_Small C21
+L Device:C_Small C21
 U 1 1 57FD814A
 P 2800 2150
@@
 $EndComp
 $Comp
-L STM32-F405RGT6 U?
+L tera_processors:STM32-F405RGT6 U?
 U 9 1 57FEF7D3
 P 3350 3250
@@
 $EndComp
 $Comp
-L STM32-F405RGT6 U?
+L tera_processors:STM32-F405RGT6 U?
 U 10 1 57FF252B
 P 3350 2150
@@
 $EndComp
 $Comp
-L Jumper_NO_Small JP4
+L Device:Jumper_NO_Small JP4
 U 1 1 58008E63
 P 2650 3000
@@
 $EndComp
 $Comp
-L LM4132A-3.3 IC1
+L Supply:LM4132A-3.3 IC1
 U 1 1 57FE0E6E
 P 1850 2050
@@
 $EndComp
 $Comp
-L Led_Small D18
+L Device:LED_Small D18
 U 1 1 5802039D
 P 5000 3300
@@
 $EndComp
 $Comp
-L R_Small R6
+L Device:R_Small R6
 U 1 1 58020C20
 P 5000 3050
@@
 $EndComp
 $Comp
-L Led_Small D19
+L Device:LED_Small D19
 U 1 1 58023967
 P 5500 3300
@@
 $EndComp
 $Comp
-L R_Small R7
+L Device:R_Small R7
 U 1 1 5802396D
 P 5500 3050
@@
 $EndComp
 $Comp
-L PWR_FLAG #FLG059
+L power:PWR_FLAG #FLG059
 U 1 1 580259B6
 P 3950 3200
@@
 $EndComp
 $Comp
-L PWR_FLAG #FLG060
+L power:PWR_FLAG #FLG060
 U 1 1 58025AC5
 P 3750 3200
@@
 $EndComp
 $Comp
-L CP_Small C28
+L Device:CP_Small C28
 U 1 1 581F45C5
 P 3950 3600
@@
 $EndComp
 $Comp
-L CP_Small C27
+L Device:CP_Small C27
 U 1 1 581F499E
 P 3750 3600
@@
 $EndComp
 $Comp
-L CP_Small C24
+L Device:CP_Small C24
 U 1 1 581F4E0F
 P 2600 2150
@@
 $EndComp
 $Comp
-L CP_Small C18
+L Device:CP_Small C18
 U 1 1 58208671
 P 1350 2050
